File: riley-penny-custom.kicad_sch (KiCad schematic)
At the start: 12 parts, among them J1 Barrel_Jack_Switch, J2 AudioJack_TRS, J3 AudioJack_TRS, Q5 Q_PMOS_GSD

Commit message: finished bd2 schematic
Parts:
- removed D8: LED, bca-footprints:LED_D5.0mm, symbol Device:LED
- removed R23: 27k, Resistor_SMD:R_0805_2012Metric_Pad1.20x1.40mm_HandSolder, symbol BCA Symbol Library:R
- added J4, J5: Conn_01x08, symbol Connector_Generic:Conn_01x08
- renumbered C15 to C1, C18 to C2, D7 to D1, FB2 to FB1, Q5 to Q1, R19 to R1
Connections:
- net Earth: now also J4.1 (Pin_1), J5.1 (Pin_1)
- net input_jack: now also J4.2 (Pin_2)
- new net bluesdriver-return: J5.3 (Pin_3)
- new net bluesdriver-send: J5.2 (Pin_2)
- new net zendrive_return: J4.4 (Pin_4)
- new net zendrive_send: J4.3 (Pin_3)
Other:
- moved on the sheet: C2, FB1
