File: zendrive.kicad_sch (KiCad schematic)
At the start: 42 parts, among them Q2 2N7000, Q3 2N7000, Q4 2N7000, SW1 SW_SPDT, U1 OPA2134, U2 DG412xY

Commit message: finished bd2 schematic
Parts:
- removed D6: BAT41, Diode_SMD:D_SOD-323_HandSoldering, symbol Device:D_Schottky
- renumbered C13 to C10, C4 to C11, C36 to C12, C37 to C13, C6 to C3, C7 to C4, C8 to C5, C9 to C6, C10 to C7, C11 to C8, C12 to C9, D2 to D3, D3 to D4, D4 to D5, FB3 to FB2, R43 to R16, R44 to R17, R4 to R3, R5 to R4, R17 to R5, U2 to U1, U1 to U2, U2 to U3, U2 to U4
Connections:
- net 9V: now also C11.1, R14.2, R15.2, U1.12 (VL), U1.13 (V+)
- net Earth: now also U1.3; no longer U1.11
- net at C4.1, C5.2, R5.2: now also U1.2; no longer U1.10
- net at C6.2, D5.2 (A), Q3.2 (G)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: now also U3.3; no longer U3.7
- net at R8.2: now also U3.2; no longer U3.6
- net V1 renamed Q1G
- net Q1G: now also U3.1; no longer U3.8
- net V2 renamed Q1D
- net Q1D: now also U1.1; no longer U1.9
Other:
- moved on the sheet: C11, C12, C13, C14, FB2, Q4, R14, R15, R16, R17, SW1, U1E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
