File: chris-mang-custom.kicad_sch (KiCad schematic)
At the start: 14 parts, among them J1 Barrel_Jack_Switch, J2 AudioJack_TRS, J3 AudioJack_TRS, J4 Conn_01x06, J5 Conn_01x06, Q1 Q_PMOS_GSD

Commit message: added bluesbreaker schematic
Connections:
- net bluesdriver-return renamed bluesbreaker-return
- net bluesdriver-send renamed bluesbreaker-send
Other:
- sheet blues-driver renamed bluesbreaker
- sheet bluesbreaker: file blues-driver.kicad_sch -> bluesbreaker.kicad_sch
- moved on the sheet: C1, C2, D1, FB1, G1, J1, J2, J3, Q1, R1, R2, R3

Commit message: first route of PCB
Other:
- moved on the sheet: C1, C2, D1, FB1, G1, J1, J2, J3, Q1, R1, R2, R3

Commit message: finalized schematic
Parts:
- R2, R3: footprint Resistor_SMD:R_0805_2012Metric_Pad1.20x1.40mm_HandSolder -> bca-footprints:R_L3.6mm_D1.6mm_P5.00mm_Horizontal
Changed lines of the file:
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@@
 			)
 		)
-		(property "Footprint" "Resistor_SMD:R_0805_2012Metric_Pad1.20x1.40mm_HandSolder"
+		(property "Footprint" "bca-footprints:R_L3.6mm_D1.6mm_P5.00mm_Horizontal"
 			(at 127 142.24 0)
 			(effects
@@
 			)
 		)
-		(property "Footprint" "Resistor_SMD:R_0805_2012Metric_Pad1.20x1.40mm_HandSolder"
+		(property "Footprint" "bca-footprints:R_L3.6mm_D1.6mm_P5.00mm_Horizontal"
 			(at 134.62 142.24 0)
 			(effects
@@
 		)
 		(instances
-			(project "riley-penny-custom"
+			(project "chris-mang-custom"
 				(path "/0931d4cd-bc79-4e0b-a395-63d6dc93deda"
 					(reference "R3")
