File: bluesbreaker.kicad_sch (KiCad schematic)
At the start: 61 parts, among them Q5 BC848C, Q6 BC848C, SW2 SW_DIP_SPDT_2pos, U3 NJM4580, U4 TLV9352

Commit message: first route of PCB
Parts:
- added R31: 100k, bca-footprints:R_L3.6mm_D1.6mm_P5.00mm_Horizontal, symbol bca-symbols:R
- C32, C33: footprint Capacitor_SMD:C_0603_1608Metric_Pad1.08x0.95mm_HandSolder -> Capacitor_SMD:C_0805_2012Metric_Pad1.18x1.45mm_HandSolder
- D10, D11, D5, D6, D7, D8, D9: footprint (none) -> bca-footprints:Diode_DO-35_P5.00mm
- Q5, Q6: footprint (none) -> Package_TO_SOT_SMD:SOT-23_Handsoldering
- RV7: value 50kA -> 100kA
- RV8, RV9: footprint bca-footprints:R_POT_9mm -> bca-footprints:R_POT
- U3: footprint (none) -> Package_SO:SOIC-8_3.9x4.9mm_P1.27mm
- renumbered R31 to R32, R32 to R33, R33 to R34, R34 to R35, R35 to R36, R36 to R37, R37 to R38, R38 to R39, R39 to R40, R40 to R41, R41 to R42, R42 to R43
Connections:
- net 4.5V: now also U3.3 (+); no longer U3.5 (+)
- net sw2: now also U3.6 (-); no longer U3.2 (-)
- net sw5: now also U3.1; no longer U3.7
- net at C18.2, RV5.2: now also U3.7; no longer U3.1
- net at R26.2, R27.1, R28.1: now also U3.2 (-); no longer U3.6 (-)
- net at C17.2, R23.2: now also U3.5 (+); no longer U3.3 (+)
- net at C21.2, RV7.1: now also R31.1
- net at R30.2, RV7.2, RV7.3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: now also R31.2
Other:
- title: Blues Driver -> Bluesbreaker w/ Clean blend
- moved on the sheet: C15, C16, C17, C18, C19, C21, C22, C23, C30, C31, C32, C33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

Commit message: finalized schematic
Parts:
- removed C24: 0.1u, bca-footprints:C_Film_L7.2mm_W2.5mm_P5.00mm, symbol bca-symbols:C_Film_W2.50mm
- removed R38: 1k, bca-footprints:R_L3.6mm_D1.6mm_P5.00mm_Horizontal, symbol bca-symbols:R
- added C24: 10u, bca-footprints:CP_Radial_D4.0mm_P1.50mm, symbol bca-symbols:CP_Audio
- C25: value 0.1u -> 47n
- C26: value 22p -> 47p
- R36: value 100k -> 180k
- R37: value 10k -> 100k
- R41: value 22k -> 10k
Connections:
- net 4.5V: now also R37.1; no longer RV8.1
- net Earth: now also RV8.1; no longer R37.1
- net return: now also RV8.2
- net at R37.2: now also C22.1, C23.1, R30.2, R31.2, RV7.2, RV7.3; no longer C27.2
- net at Q5.2 (E), R33.2: now also C24.1
- net at R34.1: now also C24.2
- new net: C27.2, RV8.3
Other:
- moved on the sheet: R37, RV8

Commit message: first draft PCB
Parts:
- added C34: 100p, bca-footprints:C_Ceramic_L4.0mm_W2.5mm_P2.50mm, symbol bca-symbols:C_Ceramic
- R24: value 10k -> 33k
- R25: value 100k -> 150k
Connections:
- net sw2: now also R24.1; no longer C18.1, R21.2, R22.2, R25.1, U3.6 (-)
- net sw7: now also C18.1, R21.2, R22.2, R25.1, U3.6 (-); no longer R24.1
- net at C25.1, RV9.2, RV9.3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: now also C34.2
- net at R41.2, RV9.1, U4.2 (-): now also C34.1
Other:
- moved on the sheet: C28, C29, Q6, R19, R39, R40, R41, RV9, U4A

Commit message: generated gerbers
Parts:
- C22: footprint bca-footprints:C_Film_L7.2mm_W3.5mm_P5.00mm -> bca-footprints:C_Film_L7.2mm_W5.00mm_P5.00mm
- R24: value 33k -> 39k
Changed lines of the file:
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@@
 			)
 		)
-		(property "Footprint" "bca-footprints:C_Film_L7.2mm_W3.5mm_P5.00mm"
+		(property "Footprint" "bca-footprints:C_Film_L7.2mm_W5.00mm_P5.00mm"
 			(at 175.26 53.6448 0)
 			(effects
@@
 			)
 		)
-		(property "Value" "33k"
+		(property "Value" "39k"
 			(at 54.61 26.416 0)
 			(effects

Commit message: re-generated gerbers, finalized BOM
Parts:
- C15, C16, C17, C20, C21, C28: value 10n -> 10nF
- C18, C34: value 100p -> 100pF
- C19: value 0.1u -> 0.1uF
- C22, C23: value 1u -> 1uF
- C24, C27, C29: value 10u -> 10uF
- C25: value 47n -> 47nF
- C26: value 47p -> 47pF
- C30, C31: value 100u -> 100uF
- C32, C33: value 100n -> 100nF
Changed lines of the file:
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@@
 			)
 		)
-		(property "Value" "100p"
+		(property "Value" "100pF"
 			(at 59.69 41.148 90)
 			(effects
@@
 			)
 		)
-		(property "Value" "100n"
+		(property "Value" "100nF"
 			(at 92.456 172.72 90)
 			(effects
@@
 			)
 		)
-		(property "Value" "1u"
+		(property "Value" "1uF"
 			(at 171.45 65.786 90)
 			(effects
@@
 			)
 		)
-		(property "Value" "10u"
+		(property "Value" "10uF"
 			(at 195.58 68.326 90)
 			(effects
@@
 			)
 		)
-		(property "Value" "10n"
+		(property "Value" "10nF"
 			(at 148.59 72.136 0)
 			(effects
@@
 			)
 		)
-		(property "Value" "10n"
+		(property "Value" "10nF"
 			(at 138.43 72.136 0)
 			(effects
@@
 			)
 		)
-		(property "Value" "10u"
+		(property "Value" "10uF"
 			(at 158.75 102.616 90)
 			(effects
@@
 			)
 		)
-		(property "Value" "10n"
+		(property "Value" "10nF"
 			(at 25.4 42.672 90)
 			(effects
@@
 			)
 		)
-		(property "Value" "1u"
+		(property "Value" "1uF"
 			(at 171.45 58.166 90)
 			(effects
@@
 			)
 		)
-		(property "Value" "100p"
+		(property "Value" "100pF"
 			(at 181.61 94.488 90)
 			(effects
@@
 			)
 		)
-		(property "Value" "100u"
+		(property "Value" "100uF"
 			(at 68.072 179.578 0)
 			(effects
@@
 			)
 		)
-		(property "Value" "100n"
+		(property "Value" "100nF"
 			(at 111.506 172.72 90)
 			(effects
@@
 			)
 		)
-		(property "Value" "0.1u"
+		(property "Value" "0.1uF"
 			(at 77.47 50.292 90)
 			(effects
@@
 			)
 		)
-		(property "Value" "47n"
+		(property "Value" "47nF"
 			(at 195.58 82.042 90)
 			(effects
@@
 			)
 		)
-		(property "Value" "47p"
+		(property "Value" "47pF"
 			(at 222.25 72.898 90)
 			(effects
@@
 			)
 		)
-		(property "Value" "10u"
+		(property "Value" "10uF"
 			(at 234.95 84.836 90)
 			(effects
@@
 			)
 		)
-		(property "Value" "100u"
+		(property "Value" "100uF"
 			(at 51.562 174.498 0)
 			(effects
@@
 			)
 		)
-		(property "Value" "10n"
+		(property "Value" "10nF"
 			(at 44.45 54.102 90)
 			(effects
@@
 			)
 		)
-		(property "Value" "10n"
+		(property "Value" "10nF"
 			(at 35.56 42.672 90)
 			(effects
@@
 			)
 		)
-		(property "Value" "10n"
+		(property "Value" "10nF"
 			(at 135.89 96.012 90)
 			(effects
